File: OtterCam-s3.kicad_pcb (KiCad board)
At the start: 4 copper layers, 49.8 x 49.8 mm, 169 parts, among them J1 UART, J2 SD, J3 USB, J4 RJ45, J5 MIPI, J6 LENS, Q1 DTA114YKA, SW1 RST, U1 AllWinner-S3(FBGA-234), U2 AXP209(QFN-48), U3 SY8089AAAC, U4 AP6236, Y1 32.768kHz, Y2 24MHz, Y3 26MHz

Commit message: new 3d files
Parts:
- removed G***: LOGO, otter:OtterCastAudioV2_hw_v2.1
- removed G***: LOGO, otter:OtterCastAudioV2_silk_1
- removed G***: LOGO, otter:OtterCastAudioV2_silk_3
- removed G***: LOGO, otter:OtterCastAudioV2_silk_amp_out
- removed G***: LOGO, otter:OtterCastAudioV2_silk_line_out
- removed G***: LOGO, otter:OtterCastAudioV2_silk_line_in
- removed G***: LOGO, otter:OtterCastAudioV2_silk_by
- removed G***: LOGO, otter:OtterCastAudioV2_silk_status
- removed G***: LOGO, otter:OtterCastAudioV2_silk_power
- removed G***: LOGO, otter:OtterCastAudioV2_silk_2
- moved R11 7.28 mm to (77.2, 65.4), turned to 270 degrees
- moved J2 0.65 mm to (80.5, 58.2), turned to 180 degrees
Routing:
- net SDC0_D2: track 6.39 -> 18.7 mm, vias 0 -> 2
- net SDC0_D1: track 8.30 -> 19.9 mm, vias 0 -> 2
- net SDC0_D3: track 7.06 -> 18.5 mm, vias 0 -> 2
- net SDC0_D0: track 7.87 -> 18.7 mm, vias 0 -> 2
- net SDC0_CMD: track 6.52 -> 17.2 mm, vias 0 -> 2
- net SDC0_CLK: track 7.27 -> 17.6 mm
- net SDC0_DET#: track 18.1 -> 11.6 mm
- net GND: track 129.9 -> 123.4 mm, vias 183 -> 234
- net Net-(C2-Pad1): track 10.8 -> 14.7 mm
- net GPIO_LED2: track 54.5 -> 55.1 mm
- net GPIO_LED1: track 51.6 -> 52.2 mm
- net +3V3: track 175.3 -> 174.9 mm, vias 25 -> 26
Other:
- board text added: "3V3"
- board text added: "GND"
- board text added: "OtterCam-s3 Jan Henrik Hemsing @JanHenrikH 2021 github.com/Jan--Henrik/OtterCam-s3"
- board text added: "RST"
- board text added: "RX"
- board text added: "TX"
- board text added: "owo"

Commit message: added all gerber
Parts:
- moved J6 3.30 mm to (66.5, 61.1)
Routing:
- net +5V: track 68.5 -> 62.9 mm, vias 4 -> 3
- net MIPI_SCK: track 102.0 -> 105.5 mm
- net MIPI_SDA: track 106.8 -> 110.2 mm
- net EPHY_LINK_LED: track 26.4 -> 27.0 mm
- net GND: vias 234 -> 233
