File: MIPI.kicad_sch (KiCad schematic)
At the start: 41 parts, among them J4 RJ45, J5 MIPI, U1 AllWinner-S3(FBGA-234), Y1 32.768kHz, Y2 24MHz

Commit message: updated hw files
Connections:
- net +1V1: now also U1.N5 (EPHY_VDD)
- net +3.0VA: now also U1.L6 (VCC_PLL), U1.M7 (AVCC)
- net +3.3V_RTC: now also U1.N6 (VCC_RTC)
- net +3V3: now also U1.M4 (VCC_MCSI), U1.M5 (EPHY_VCC), U1.N7 (VCC_USB), U1.P12 (HPVCCIN)
- net AP_CK32KO: now also U1.P3 (X32KFOUT)
- net EPHY_LINK_LED: now also U1.K5 (EPHY_LINK_LED)
- net EPHY_RX_N: now also U1.F1 (EPHY_RXN)
- net EPHY_RX_P: now also U1.F2 (EPHY_RXP)
- net EPHY_SPD_LED: now also U1.L5 (EPHY_SPD_LED)
- net EPHY_TX_N: now also U1.E2 (EPHY_TXN)
- net EPHY_TX_P: now also U1.E3 (EPHY_TXP)
- net GND: now also U1.P8 (AGND)
- net LRADC0: now also U1.T8 (LRADC0)
- net LRADC1: now also U1.R8 (LRADC1)
- net MIPI_CK_N: now also U1.J1 (MCSI_CKN)
- net MIPI_CK_P: now also U1.J2 (MCSI_CKP)
- net MIPI_D0_N: now also U1.G2 (MCSI_D0N)
- net MIPI_D0_P: now also U1.G3 (MCSI_D0P)
- net MIPI_D1_N: now also U1.H1 (MCSI_D1N)
- net MIPI_D1_P: now also U1.H2 (MCSI_D1P)
- net MIPI_D2_N: now also U1.K1 (MCSI_D2N)
- net MIPI_D2_P: now also U1.K2 (MCSI_D2P)
- net MIPI_D3_N: now also U1.L2 (MCSI_D3N)
- net MIPI_D3_P: now also U1.L3 (MCSI_D3P)
- net NMI: now also U1.R7 (NMI)
- net RESETn: now also U1.P7 (RESET)
- net USB_D_N: now also U1.R2 (USB_DM)
- net USB_D_P: now also U1.T2 (USB_DP)
- net at C50.1, R47.1: now also U1.N10 (VRA2)
- net at R55.2: now also U1.P6 (EPHY_RTX); no longer U1.A2 (PB13/JTAG_DI/PB_EINT13)
- net at R50.1: now also U1.R13 (JTAG_SEL)
- net at C53.1: now also U1.M9 (HPVCCBP)
- net at C51.1, C52.1, C54.1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: now also U1.H6 (DVREF)
- net at R51.1: now also U1.J5 (DZQ)
- net at R52.1: now also U1.F5 (ZQ)
- net at C58.1, Y2.1: now also U1.R4 (X24MIN)
- net at C59.1, Y2.3: now also U1.P4 (X24MOUT)
- net at C56.1: now also U1.T5 (RTC_VIO)
- net at C61.1, R53.2, Y1.1: now also U1.T3 (X32KIN)
- net at C62.1, R53.1, Y1.2: now also U1.R3 (X32KOUT)

Commit message: updated schematic files
Other:
- company: (none) -> Jana Marie Hemsing
- title: OtterCastAudioV2 -> OtterCamS3
Changed lines of the file:
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@@
   (paper "A4")
   (title_block
-    (title "OtterCastAudioV2")
+    (title "OtterCamS3")
+    (date "2023-02-02")
     (rev "1.0")
+    (company "Jana Marie Hemsing")
   )
   (junction (at 123.19 111.76) (diameter 0) (color 0 0 0 0)
