File: Power.kicad_sch (KiCad schematic)
At the start: 70 parts, among them J3 USB, Q1 DTA114YKA, SW1 RST, U1 AllWinner-S3(FBGA-234), U2 AXP209(QFN-48), U3 SY8089AAAC

Commit message: updated schematic files
Connections:
- net +1V1: now also U1.G12 (VDD_CPU0), U1.H12 (VDD_CPU1), U1.J11 (VDD_CPU2), U1.J12 (VDD_CPU3), U1.K11 (VDD_CPU4), U1.K8 (VDD_SYS0), U1.K9 (VDD_SYS1), U1.L8 (VDD_SYS2), U1.M8 (VDD_SYS3); no longer U1.A7 (PB6/TWI0_SCK/PB_EINT6), U1.B3 (PB0/UART2_TX/PB_EINT0), U1.B8 (PB2/UART2_RTS/PB_EINT2), U1.C4 (PB3/UART2_CTS/PB_EINT3), U1.C7 (PB5/PWM1/PB_EINT5), U1.C8 (PB4/PWM0/PB_EINT4)
- net +3V3: now also U1.H11 (VCC_IO0), U1.P5 (VCC_IO1)
- net GND: now also U1.D10 (GND29), U1.D11 (GND30), U1.D12 (GND31), U1.D6 (GND25), U1.D8 (GND27), U1.D9 (GND28), U1.E14 (GND0), U1.E4 (GND32), U1.E5 (GND33), U1.E6 (GND34), U1.E7 (GND35), U1.E8 (GND36), U1.E9 (GND37), U1.F10 (GND2), U1.J4 (GND18), U1.J7 (GND58), U1.N4 (GND43); no longer U1.A2 (PB13/JTAG_DI/PB_EINT13), U1.A3 (PC0/SDC2_CLK/SPI0_MISO), U1.B1 (PC2/SDC2_RST/SPI0_CS), U1.B2 (PC1/SDC2_CMD/SPI0_CLK), U1.C1 (PC6/SDC2_D3), U1.C2 (PC3/SDC2_D0/SPI0_MOSI), U1.C3 (PC7/SDC2_D4), U1.D1 (PC10/SDC2_D7), U1.D2 (PC9/SDC2_D6), U1.D3 (PC8/SDC2_D5), U1.F3 (PC4/SDC2_D1), U1.F4 (PC5/SDC2_D2)
- net VCC-DDR: now also U1.F6 (VCC_DRAM0), U1.F7 (VCC_DRAM1), U1.F8 (VCC_DRAM2), U1.G8 (VCC_DRAM3), U1.H8 (VCC_DRAM4), U1.J8 (VCC_DRAM5); no longer U1.A5 (PB10/JTAG_MS/PB_EINT10), U1.B5 (PB12/JTAG_DO/PB_EINT12), U1.B6 (PB8/TWI1_SCK/UART0_TX/PB_EINT8), U1.C5 (PB11/JTAG_CK/PB_EINT11), U1.C6 (PB9/TWI1_SDA/UART0_RX/PB_EINT9)
- net at R31.1: now also U1.M6 (VDD_EFUSE)
Other:
- company: (none) -> Jana Marie Hemsing
- title: OtterCastAudioV2 -> OtterCamS3
Changed lines of the file:
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@@
   (paper "A3")
   (title_block
-    (title "OtterCastAudioV2")
+    (title "OtterCamS3")
+    (date "2023-02-02")
     (rev "1.0")
+    (company "Jana Marie Hemsing")
   )
   (junction (at 262.89 96.52) (diameter 0) (color 0 0 0 0)
@@
     (pin "9")
   )
-  (symbol (lib_id "otter:AllWinner-S3(FBGA-234)") (at 323.85 99.06 0) (unit 1)
+  (symbol (lib_id "otter:AllWinner-S3(FBGA-234)") (at 323.85 99.06 0) (unit 4)
     (in_bom yes) (on_board yes)
     (property "Reference" "U1" (id 0) (at 323.85 56.3626 0))
@@
       (effects (font (size 1.27 1.27)) hide)
     )
-    (pin "A2")
-    (pin "A3")
-    (pin "A5")
-    (pin "A7")
-    (pin "B1")
-    (pin "B2")
-    (pin "B3")
-    (pin "B4")
-    (pin "B5")
-    (pin "B6")
-    (pin "B7")
-    (pin "B8")
-    (pin "C1")
-    (pin "C2")
-    (pin "C3")
-    (pin "C4")
-    (pin "C5")
-    (pin "C6")
-    (pin "C7")
-    (pin "C8")
-    (pin "D1")
-    (pin "D2")
-    (pin "D3")
-    (pin "F3")
-    (pin "F4")
+    (pin "A1")
+    (pin "A16")
+    (pin "C9")
+    (pin "D10")
+    (pin "D11")
+    (pin "D12")
+    (pin "D4")
+    (pin "D5")
+    (pin "D6")
+    (pin "D7")
+    (pin "D8")
+    (pin "D9")
+    (pin "E10")
+    (pin "E11")
+    (pin "E14")
+    (pin "E4")
+    (pin "E5")
+    (pin "E6")
+    (pin "E7")
+    (pin "E8")
+    (pin "E9")
+    (pin "F10")
+    (pin "F11")
+    (pin "F6")
+    (pin "F7")
+    (pin "F8")
+    (pin "F9")
+    (pin "G10")
+    (pin "G11")
+    (pin "G12")
+    (pin "G4")
+    (pin "G5")
+    (pin "G6")
+    (pin "G7")
+    (pin "G8")
+    (pin "G9")
+    (pin "H10")
+    (pin "H11")
+    (pin "H12")
+    (pin "H3")
+    (pin "H4")
+    (pin "H5")
+    (pin "H7")
+    (pin "H8")
+    (pin "H9")
+    (pin "J10")
+    (pin "J11")
+    (pin "J12")
+    (pin "J3")
+    (pin "J4")
+    (pin "J6")
+    (pin "J7")
+    (pin "J8")
+    (pin "J9")
+    (pin "K10")
+    (pin "K11")
+    (pin "K12")
+    (pin "K3")
+    (pin "K4")
+    (pin "K6")
+    (pin "K7")
+    (pin "K8")
+    (pin "K9")
+    (pin "L10")
+    (pin "L4")
+    (pin "L7")
+    (pin "L8")
+    (pin "L9")
+    (pin "M10")
+    (pin "M6")
+    (pin "M8")
+    (pin "N4")
+    (pin "N8")
+    (pin "P5")
+    (pin "R5")
+    (pin "T1")
+    (pin "T16")
   )
   (symbol (lib_id "Device:R_Small") (at 307.34 220.98 180) (unit 1)
