File: WifiBT.kicad_sch (KiCad schematic)
At the start: 26 parts, among them U4 AP6236, Y3 26MHz

Commit message: updated schematic files
Other:
- company: (none) -> Jana Marie Hemsing
- title: OtterCastAudioV2 -> OtterCamS3
Changed lines of the file:
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@@
   (paper "A4")
   (title_block
-    (title "OtterCastAudioV2")
+    (title "OtterCamS3")
+    (date "2023-02-02")
     (rev "1.0")
+    (company "Jana Marie Hemsing")
   )
   (junction (at 190.5 85.09) (diameter 0) (color 0 0 0 0)
