File: lensmount_v1.0/lensmount-v1.0.kicad_pcb (KiCad board)
At the start: 2 copper layers, 49.8 x 49.8 mm, 43 parts, among them J1 VBAT, J10 Picoblade DNP, J2 DETECT, J3 AGND, J4 VDD, J5 DOUT, J6 DIN, J7 DCLK, J8 DGND, P1 TC2030-CTX-Tag-Connect, Q1 2N7002, Q2 2N7002, Q3 2N7002, Q4 AO3401A, Q5 AO3401A, U1 STM32F042F6Px, U2 XC6206PxxxMR, U3 USBLC6-4

Commit message: added all gerber
Parts:
- removed C5: 100n, otter:C_0402
- removed R1, R2: 5k1, otter:R_0402
- removed U3: USBLC6-4, Package_TO_SOT_SMD:SOT-23-6
- P1: moved to F.Cu
- U1: value STM32F042F6Px -> STM32F042G6Ux; footprint Package_SO:TSSOP-20_4.4x6.5mm_P0.65mm -> Package_DFN_QFN:QFN-28_4x4mm_P0.5mm
- moved C2 55.0 mm to (122.9, 83.5), turned to 180 degrees
- moved C1 51.2 mm to (118.0, 87.2), turned to 270 degrees
- moved P1 48.5 mm to (114.7, 78.9), turned to 90 degrees
- moved C4 47.6 mm to (112.3, 78.3), turned to 90 degrees
- moved R3 46.6 mm to (122.7, 114.7), turned to 270 degrees
- moved R5 45.8 mm to (122.7, 111.2), turned to 270 degrees
- moved U2 44.3 mm to (110.0, 78.1), turned to 180 degrees
- moved C3 42.7 mm to (107.6, 77.3), turned to 90 degrees
- moved Q1 42.2 mm to (120.5, 114.6), turned to 180 degrees
- moved U1 41.9 mm to (121.1, 86.6), turned to 180 degrees
- moved R4 41.8 mm to (114.3, 122.3), turned to 225 degrees
- moved Q3 41.4 mm to (120.5, 111.1), turned to 180 degrees
- moved C6 41.0 mm to (90.0, 122.7), turned to 0 degrees
- moved Q2 37.8 mm to (112.8, 120.7), turned to 135 degrees
- moved Q4 36.2 mm to (89.0, 120.2)
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Connections:
- J10 pad 1: GND -> VBUS
- J10 pad 2: VBUS -> SDA
- J10 pad 3: UART_RX -> SCK
- J10 pad 4: UART_TX -> GND
- U1 pad 14: Net-(U1-Pad14) -> EN_VBAT
- U1 pad 15: GND -> EN_VBUS
- U1 pad 16: +3V3 -> GND
- U1 pad 17: D- -> +3V3
- U1 pad 18: D+ -> +3V3
- U1 pad 19: SWDIO -> SCK
- U1 pad 2: EN_VBAT -> Net-(U1-Pad2)
- U1 pad 20: SWCLK -> SDA
- U1 pad 3: EN_VBUS -> Net-(U1-Pad3)
- U1 pad 8: UART_TX -> Net-(U1-Pad8)
- U1 pad 9: UART_RX -> Net-(U1-Pad9)
Routing:
- net VBUS: track 40.6 -> 124.5 mm, vias 3 -> 0
- net DETECT: track 9.20 -> 88.3 mm, vias 0 -> 1
- net EN_VBUS: track 0.00 -> 76.4 mm, vias 0 -> 2
- net +3V3: track 0.00 -> 72.1 mm, vias 1 -> 2
- net EN_VBAT: track 14.6 -> 75.8 mm
- net DOUT_3V3: track 0.00 -> 40.2 mm
- net UART_TX: track 39.0 -> 0.00 mm, vias 2 -> 0
- net SCK: track 0.00 -> 38.8 mm
- net SDA: track 0.00 -> 37.6 mm
- net DIN_3V3: track 0.00 -> 31.5 mm, vias 0 -> 2
- net GND: track 4.70 -> 32.2 mm, vias 23 -> 35
- net DCLK_3V3: track 0.00 -> 26.8 mm
- net DIN_5V: track 3.80 -> 21.4 mm, vias 0 -> 1
- net Net-(J4-Pad1): track 0.00 -> 17.0 mm, vias 0 -> 2
- net DOUT_5V: track 0.00 -> 15.4 mm, vias 0 -> 1
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- removed copper zone on B.Cu, net VBUS
Other:
- board text added: "@JanHenrikH 2021 github.com/Jan--Henrik/OtterCam-s3"
- board text added: "OtterCam-s3 Lensmount EF(-S) Jan Henrik Hemsing"
