File: sensor_OS05A10_A20/sensor.kicad_sch (KiCad schematic)
At the start: 41 parts, among them J1 FH35C-25S, U1 LP2985-2.8, U2 LP2985-1.8, U3 LP2985-1.2, U4 OS05A10-SMU

Commit message: updated sensor board
Other:
- company: (none) -> Jana Marie Hemsing
- title: (none) -> OS05A10/OS05A20 Sensor board
Changed lines of the file:
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@@
 (kicad_sch (version 20211123) (generator eeschema)
   (paper "A4")
+  (title_block
+    (title "OS05A10/OS05A20 Sensor board")
+    (date "2023-02-02")
+    (rev "v1.1.1")
+    (company "Jana Marie Hemsing")
+  )
   (junction (at 172.72 95.25) (diameter 0) (color 0 0 0 0)
   )
