File: lensmount_efs/lensmount.kicad_sch (KiCad schematic)
At the start: 38 parts, among them J1 VBAT, J10 Picoblade DNP, J2 DETECT, J3 AGND, J4 VDD, J5 DOUT, J6 DIN, J7 DCLK, J8 DGND, P1 TC2030-CTX-Tag-Connect, Q1 2N7002, Q2 2N7002, Q3 2N7002, Q4 AO3401A, Q5 AO3401A, U1 STM32F042G6Ux, U2 XC6206PxxxMR

Commit message: updated lensmount
Other:
- company: (none) -> Jana Marie hemsing
- title: (none) -> EF-S Mount board
Changed lines of the file:
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@@
 (kicad_sch (version 20211123) (generator eeschema)
   (paper "A4")
+  (title_block
+    (title "EF-S Mount board")
+    (date "2023-02-02")
+    (rev "v1.0.1")
+    (company "Jana Marie hemsing")
+  )
   (junction (at 176.53 135.89) (diameter 0) (color 0 0 0 0)
   )
